File: Schaltpläne/Stratoballon/Stratoballon.sch (KiCad schematic (older format))
At the start: 7 parts, among them J1 Conn_02x20_Top_Bottom_Mountin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

Commit message: Schaltpläne bearbeitet * ToDo Liste angelegt * Sensoren teilweise eingefügt
Parts:
- added B2: BMP280, Package_LGA:Bosch_LGA-8_2x2.5mm_P0.65mm_ClockwisePinNumbering, symbol Sensor_Pressure:BMP280
- added C5: 0,33µF, symbol Device:C
- added J2: Conn_01x03_Female, symbol Connector:Conn_01x03_Female
- gave numbers to parts that had none: 1
Connections:
- wire segments 115 -> 137
Other:
- note added: "Anschluss für\nGeigerzähler"
- moved on the sheet: A1, B1, C2, C3, C4, D1, J1
